Commit message: 6.2.6贴合地面，添加虚拟部件（影子）

File: install/my_robo_description/share/my_robo_description/URDF/base.urdf.xacro (robot description, xacro)
@@ -3,4 +3,6 @@
     <!-- 定义 base_link 宏 -->
     <xacro:macro name="base_xacro" params="length radius">
+        <!--机器人的影子-->
+        <link name="base_foot_print_yingzi" />
         <!-- 机器人的身体部分 -->
         <link name="base_link">
@@ -21,4 +23,9 @@
             </visual>
         </link>
+        <joint name="base_joint" type="fixed">
+            <origin xyz="0.0 0.0 ${length/2.0+0.032-0.001}" rpy="0.0 0.0 0.0"/>
+            <parent link="base_foot_print_yingzi"/>
+            <child link="base_link"/>
+        </joint>
     </xacro:macro>
 </robot>

Commit message: 6.3.1 添加碰撞属性

File: install/my_robo_description/share/my_robo_description/URDF/base.urdf.xacro (robot description, xacro)
@@ -22,4 +22,18 @@
                 </material>
             </visual>
+            <collision>
+                 <!-- 沿着自己几何中心的偏移旋转量 -->
+                <origin xyz="0.0 0.0 0.0" rpy="0.0 0.0 0.0"/>
+                <!-- 几何形状 -->
+                <geometry>
+                    <!-- 圆柱体 半径0.1 高度 0.12 -->
+                    <cylinder radius="${radius}" length="${length}"/>
+                </geometry>
+                <!-- 材质 颜色描述 -->
+                <material name="white">
+                    <!-- 设置透明为 0.5 -->
+                    <color rgba="1.0 1.0 1.0 0.5"/>
+                </material>
+            </collision>
         </link>
         <joint name="base_joint" type="fixed">

File: install/my_robo_description/share/my_robo_description/URDF/body_/wheel.urdf.xacro (robot description, xacro)
@@ -20,4 +20,18 @@
                 </material>
             </visual>
+            <collision>
+                <!-- 沿着自己几何中心的偏移旋转量 -->
+                <origin xyz="0.0 0.0 0.0" rpy="1.57079 0.0 0.0"/>
+                <!-- 几何形状 -->
+                <geometry>
+                    <!-- box 自己自动生成的 正方体 -->
+                    <cylinder radius="0.032" length="0.04"/>
+                </geometry>
+                <!-- 材质 颜色描述 -->
+                <material name="yellow">
+                    <!-- 设置透明为 0.5 -->
+                    <color rgba="1.0 1.0 0.0 0.8"/>
+                </material>
+            </collision>
         </link>
         <!-- 机器人的关节 用于组合机器人的部件 -->

File: install/my_robo_description/share/my_robo_description/URDF/body_/wheel_wangxianglun.urdf.xacro (robot description, xacro)
@@ -20,4 +20,18 @@
                 </material>
             </visual>
+            <collision>
+                <!-- 沿着自己几何中心的偏移旋转量 -->
+                <origin xyz="0.0 0.0 0.0" rpy="0.0 0.0 0.0"/>
+                <!-- 几何形状 -->
+                <geometry>
+                    <!-- box 自己自动生成的 正方体 -->
+                    <sphere radius="0.016"/>  <!--球体 半径为0.016-->
+                </geometry>
+                <!-- 材质 颜色描述 -->
+                <material name="yellow">
+                    <!-- 设置透明为 0.5 -->
+                    <color rgba="0.5 1.0 0.2 0.8"/>
+                </material>
+            </collision>
         </link>
         <!-- 机器人的关节 用于组合机器人的部件 -->

File: install/my_robo_description/share/my_robo_description/URDF/sensor/camera.urdf.xacro (robot description, xacro)
@@ -20,4 +20,18 @@
                 </material>
             </visual>
+            <collision>
+                 <!-- 沿着自己几何中心的偏移旋转量 -->
+                <origin xyz="0.0 0.0 0.0" rpy="0.0 0.0 0.0"/>
+                <!-- 几何形状 -->
+                <geometry>
+                    <!-- box 自己自动生成的 正方体 -->
+                    <box size="0.02 0.02 0.02"/>
+                </geometry>
+                <!-- 材质 颜色描述 -->
+                <material name="red">
+                    <!-- 设置透明为 0.5 -->
+                    <color rgba="1.0 0.0 0.0 0.5"/>
+                </material>
+            </collision>
         </link>
         <!-- 机器人的关节 用于组合机器人的部件 -->

File: install/my_robo_description/share/my_robo_description/URDF/sensor/imu.urdf.xacro (robot description, xacro)
@@ -20,4 +20,19 @@
                 </material>
             </visual>
+            <!--增加碰撞属性-->
+            <collision>
+                     <!-- 沿着自己几何中心的偏移旋转量 -->
+                <origin xyz="0.0 0.0 0.0" rpy="0.0 0.0 0.0"/>
+                <!-- 几何形状 -->
+                <geometry>
+                    <!-- box 自己自动生成的 正方体 -->
+                    <box size="0.02 0.02 0.02"/>
+                </geometry>
+                <!-- 材质 颜色描述 -->
+                <material name="red">
+                    <!-- 设置透明为 0.5 -->
+                    <color rgba="1.0 0.0 0.0 0.5"/>
+                </material>
+            </collision>
         </link>
         <!-- 机器人的关节 用于组合机器人的部件 -->

File: install/my_robo_description/share/my_robo_description/URDF/sensor/lidar.urdf.xacro (robot description, xacro)
@@ -19,4 +19,19 @@
                 </material>
             </visual>
+            <!--增加碰撞属性-->
+            <collision>
+                <!-- 沿着自己几何中心的偏移旋转量 -->
+                <origin xyz="0.0 0.0 0.0" rpy="0.0 0.0 0.0"/>
+                <!-- 几何形状 -->
+                <geometry>
+                    <!-- box 自己自动生成的 正方体 -->
+                    <cylinder radius="0.01" length="0.10"/>
+                </geometry>
+                <!-- 材质 颜色描述 -->
+                <material name="green">
+                    <!-- 设置透明为 0.5 -->
+                    <color rgba="1.0 0.2 0.0 0.8"/>
+                </material>
+            </collision>
         </link>
         <!-- 雷达 -->
@@ -37,4 +52,19 @@
                 </material>
             </visual>
+            <!--增加碰撞属性-->
+            <collision>
+                <!-- 沿着自己几何中心的偏移旋转量 -->
+                <origin xyz="0.0 0.0 0.0" rpy="0.0 0.0 0.0"/>
+                <!-- 几何形状 -->
+                <geometry>
+                    <!-- box 自己自动生成的 正方体 -->
+                    <cylinder radius="0.02" length="0.02"/>
+                </geometry>
+                <!-- 材质 颜色描述 -->
+                <material name="yellow">
+                    <!-- 设置透明为 0.5 -->
+                    <color rgba="1.0 0.0 0.0 1.0"/>
+                </material>
+            </collision>
         </link>
         <!-- 机器人的关节 用于组合机器人的部件 -->
